File: Motor Driver PCB/MotorDriver/MotorDriver.sch (KiCad schematic (older format))
At the start: 48 parts, among them IC1 DRV8837CDSGR, IC2 DRV8837CDSGR, IC3 DRV8837CDSGR, IC4 DRV8837CDSGR, J1 M1, J10 Conn_01x04_Female, J2 M4, J3 M3, J4 M2, J5 Front vl106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

Commit message: MotorDriverRev2
New PCB design. Correct numerous errors.
Other:
- note added: "GPIO 34 -39 cannot generate PWM?"
Changed lines of the file:
@@
 Text Notes 3300 2800 0    50   ~ 0
 Connected to Intigrated SPI Flash
+Text Notes 3800 3200 0    50   ~ 0
+GPIO 34 -39 cannot generate PWM?
 $EndSCHEMATC
