File: Motor Driver PCB/MotorDriverRev2/MotorDriver.sch (KiCad schematic (older format))
At the start: 48 parts, among them IC1 DRV8837CDSGR, IC2 DRV8837CDSGR, IC3 DRV8837CDSGR, IC4 DRV8837CDSGR, J1 M1, J10 Conn_01x04_Female, J2 M4, J3 M3, J4 M2, J5 Front vl106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

Commit message: MotorDriverRev2
New PCB design. Correct numerous errors.
Parts:
- removed C37: 100uf, Capacitor_SMD:C_1206_3216Metric, symbol Device:C_Small
- removed J10: Conn_01x04_Female, Connector_PinHeader_2.00mm:PinHeader_1x05_P2.00mm_Vertical, symbol Connector:Conn_01x04_Female
- removed J6: right vl106, Connector_PinHeader_2.00mm:PinHeader_1x04_P2.00mm_Vertical, symbol Connector_Generic_Shielded:Conn_01x04_Shielded
- removed J7: leftVl106, Connector_PinHeader_2.00mm:PinHeader_1x04_P2.00mm_Vertical, symbol Connector_Generic_Shielded:Conn_01x04_Shielded
- removed U2, U5: MIC5216-3.3BM5-TR, LDO - MIC521633BM5TR:MIC5216-3.3BM5-TR, symbol 2020-07-16_00-29-16:MIC5216-3.3BM5-TR
- added C18: 10uF, Capacitor_SMD:C_0402_1005Metric, symbol Device:C_Small
- added C19: 0.1uf, Capacitor_SMD:C_0402_1005Metric, symbol Device:C_Small
- added IC5: ISL9110IRT7Z-T7A, SamacSys_Parts:SON40P300X300X75-13N, symbol SamacSys_Parts:ISL9110IRT7Z-T7A
- added J10: IO, Connector_PinHeader_2.00mm:PinHeader_1x02_P2.00mm_Vertical, symbol Connector:Conn_01x02_Female
- added L1: 2.2 uH, SamacSys_Parts:LQH3NPN100MMEL, symbol pspice:INDUCTOR
- added R3, R4: 4.7k, Resistor_SMD:R_0402_1005Metric, symbol Device:R_Small_US
- added U2: BMP280, Package_LGA:Bosch_LGA-8_2x2.5mm_P0.65mm_ClockwisePinNumbering, symbol Sensor_Pressure:BMP280
- C6: value 100uf -> 10uF; footprint Capacitor_SMD:C_1206_3216Metric -> Capacitor_SMD:C_0402_1005Metric
- J5: value Front vl106 -> I2C
- J9: value Conn_01x04_Female -> Uart; footprint Connector_PinHeader_2.00mm:PinHeader_1x05_P2.00mm_Vertical -> Connector_PinHeader_2.00mm:PinHeader_1x04_P2.00mm_Vertical
- JP1: value Jumper_NO_Small -> RST
- JP2: value Jumper_NO_Small -> BOOT
Connections:
- net labels added: IO34, IO35, UWB_RST, VBAT
- net labels removed: IO12, IO25, IO5, VBUS, VM
- wire segments 210 -> 237
- no-connect marks 6 -> 7
Other:
- note added: "GPIO 34 -39 cannot generate PWM?"
